File: pcbs/karn-right/_autosave-karn-right.kicad_sch (KiCad schematic)
At the start: 45 parts, among them J1 S2B-PH-K-SLFSN, SW11 SW_Push, SW12 SW_Push, SW13 SW_Push, SW14 SW_Push, SW15 SW_Push, SW21 SW_Push, SW22 SW_Push, SW23 SW_Push, SW24 SW_Push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

Commit message: Various changes:
- Fix incorrect reset-switch-TL3313 symbol and footprint
- Increase size of diode footprint pads
Parts:
- RSW1: footprint TL3313AF250QG_EWI -> karn-kicad:reset-switch-TL3313AF250QG
Changed lines of the file:
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@@
       (effects (font (size 1.27 1.27)) hide)
     )
-    (property "Footprint" "TL3313AF250QG_EWI" (id 2) (at 224.2785 94.8773 0)
+    (property "Footprint" "karn-kicad:reset-switch-TL3313AF250QG" (id 2) (at 224.2785 94.8773 0)
       (effects (font (size 1.524 1.524)) hide)
     )
@@
   (symbol (lib_id "power:GND") (at 214.2785 86.8773 270) (unit 1)
     (in_bom yes) (on_board yes)
-    (property "Reference" "#PWR?" (id 0) (at 207.9285 86.8773 0)
+    (property "Reference" "#PWR0101" (id 0) (at 207.9285 86.8773 0)
       (effects (font (size 1.27 1.27)) hide)
     )
@@
     )
     (path "/e3a47704-cb4a-4555-aa4f-d3ca75c136b6"
-      (reference "#PWR?") (unit 1) (value "GND") (footprint "")
+      (reference "#PWR0101") (unit 1) (value "GND") (footprint "")
     )
     (path "/817acd3d-65d5-4d98-84f9-5556e4094c7a"
@@
     )
     (path "/0eece0c9-6947-4883-a87e-b445b80630d9"
-      (reference "RSW1") (unit 1) (value "SW_Push") (footprint "TL3313AF250QG_EWI")
+      (reference "RSW1") (unit 1) (value "SW_Push") (footprint "karn-kicad:reset-switch-TL3313AF250QG")
     )
     (path "/60c85a9c-c0d2-4469-b84c-2eacd924bd6c"
