File: pcbs/karn-left/karn-left.kicad_sch (KiCad schematic)
At the start: 42 parts, among them J1 S2B-PH-K-SLFSN, SW11 SW_Push, SW12 SW_Push, SW13 SW_Push, SW14 SW_Push, SW15 SW_Push, SW21 SW_Push, SW22 SW_Push, SW23 SW_Push, SW24 SW_Push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

Commit message: Update karn-left pcb
- Apply various fixes from lessons learned on karn-right
- Fix incorrectly oriented reset switch
- Swap incorrect default polarity of JST connector footprint
- Increase size of diode pads
Parts:
- J1: footprint kbd:S2B-PH-K-SLFSN -> karn-kicad:battery-connector-S2B-PH-K-SLFSN
Connections:
- net GND: now also RSW1.4
- net reset: now also RSW1.1; no longer RSW1.2
- no-connect marks 14 -> 13
Changed lines of the file:
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@@
   (no_connect (at 188.0872 72.9089))
   (no_connect (at 174.1172 103.3889))
-  (no_connect (at 214.2785 86.8773))
   (no_connect (at 228.9292 66.2603))
-  (no_connect (at 232.2785 86.8773))
+  (no_connect (at 232.2785 90.8773))
   (no_connect (at 152.5272 90.6889))
   (no_connect (at 152.5272 88.1489))
@@
     (pin "1")
     (pin "2")
+  )
+  (symbol (lib_id "power:GND") (at 214.2785 86.8773 270) (unit 1)
+    (in_bom yes) (on_board yes)
+    (property "Reference" "#PWR0101" (id 0) (at 207.9285 86.8773 0)
+      (effects (font (size 1.27 1.27)) hide)
+    )
+    (property "Value" "GND" (id 1) (at 210.4685 86.8773 0))
+    (property "Footprint" "" (id 2) (at 214.2785 86.8773 0)
+      (effects (font (size 1.27 1.27)) hide)
+    )
+    (property "Datasheet" "" (id 3) (at 214.2785 86.8773 0)
+      (effects (font (size 1.27 1.27)) hide)
+    )
+    (pin "1")
   )
   (symbol (lib_name "D_15") (lib_id "Device:D") (at 106.4739 91.6582 270) (mirror x) (unit 1)
@@
     (pin "2")
   )
-  (symbol (lib_id "power:GND") (at 232.2785 90.8773 90) (unit 1)
-    (in_bom yes) (on_board yes)
-    (property "Reference" "#PWR05" (id 0) (at 238.6285 90.8773 0)
-      (effects (font (size 1.27 1.27)) hide)
-    )
-    (property "Value" "GND" (id 1) (at 236.0885 90.8773 0))
-    (property "Footprint" "" (id 2) (at 232.2785 90.8773 0)
-      (effects (font (size 1.27 1.27)) hide)
-    )
-    (property "Datasheet" "" (id 3) (at 232.2785 90.8773 0)
+  (symbol (lib_id "power:GND") (at 232.2785 86.8773 90) (unit 1)
+    (in_bom yes) (on_board yes)
+    (property "Reference" "#PWR05" (id 0) (at 238.6285 86.8773 0)
+      (effects (font (size 1.27 1.27)) hide)
+    )
+    (property "Value" "GND" (id 1) (at 236.0885 86.8773 0))
+    (property "Footprint" "" (id 2) (at 232.2785 86.8773 0)
+      (effects (font (size 1.27 1.27)) hide)
+    )
+    (property "Datasheet" "" (id 3) (at 232.2785 86.8773 0)
       (effects (font (size 1.27 1.27)) hide)
     )
@@
       (effects (font (size 1.524 1.524)) (justify left))
     )
-    (property "Footprint" "kbd:S2B-PH-K-SLFSN" (id 2) (at 264.6491 67.2658 0)
+    (property "Footprint" "karn-kicad:battery-connector-S2B-PH-K-SLFSN" (id 2) (at 264.6491 67.2658 0)
       (effects (font (size 1.524 1.524)) hide)
     )
@@
       (reference "#PWR09") (unit 1) (value "VCC") (footprint "")
     )
+    (path "/400bae89-5d7c-4789-ba63-752502322699"
+      (reference "#PWR0101") (unit 1) (value "GND") (footprint "")
+    )
     (path "/817acd3d-65d5-4d98-84f9-5556e4094c7a"
       (reference "D11") (unit 1) (value "D") (footprint "Diode_SMD:1N4148X-TP")
@@
     )
     (path "/a53ef69a-8078-4623-9cd4-3672c42f5863"
-      (reference "J1") (unit 1) (value "S2B-PH-K-SLFSN") (footprint "kbd:S2B-PH-K-SLFSN")
+      (reference "J1") (unit 1) (value "S2B-PH-K-SLFSN") (footprint "karn-kicad:battery-connector-S2B-PH-K-SLFSN")
     )
     (path "/0eece0c9-6947-4883-a87e-b445b80630d9"
