File: pcbs/karn-2/karn-2.kicad_pcb (KiCad board)
At the start: 2 copper layers, 139.2 x 98 mm, 23 parts, among them J1 TRRS, K11 SW_Push, K12 SW_Push, K13 SW_Push, K14 SW_Push, K15 SW_Push, K21 SW_Push, K22 SW_Push, K23 SW_Push, K24 SW_Push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

Commit message: Add karn-2 gerber files
Connections:
- U1 pad 38: VCC -> (no net)
- U2 pad 38: VCC -> (no net)
Routing:
- net /TX: track 0.00 -> 49.5 mm
- net /RX: track 0.00 -> 47.5 mm
- net /K25: track 101.4 -> 147.8 mm
- net /K24: track 81.7 -> 117.0 mm
- net VCC: track 0.00 -> 30.5 mm
- net /K11: track 18.2 -> 37.2 mm
- net /K34: track 81.1 -> 100.0 mm
- net /K13: track 54.8 -> 73.7 mm
- net /K32: track 39.4 -> 58.3 mm
- net /K31: track 20.9 -> 39.8 mm
- net /K12: track 36.8 -> 55.6 mm
- net /K35: track 100.9 -> 119.6 mm
- net /K33: track 60.9 -> 79.7 mm
- net /K15: track 92.8 -> 111.6 mm
- net /K14: track 72.8 -> 91.6 mm
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Other:
- board text added: "robcmills/karn-keyboard"
